Commit message: 添加了激光雷达模型文件

File: libro_model/urdf/gazebo_conf.xacro (robot description, xacro)
@@ -1,4 +1,20 @@
 <?xml version="1.0"?>
 <robot>
+  <!-- Add transmission to each wheel joint -->
+  <macro name="wheel_trans" params="prefix_name">
+    <transmission name="${prefix_name}_wheel_transmission">
+      <type>transmission_interface/SimpleTransmission</type>
+      <joint name="${prefix_name}_wheel_joint">
+        <hardwareInterface>hardware_interface/VelocityJointInterface</hardwareInterface>
+      </joint>
+      <actuator name="${prefix_name}_wheel_motor">
+        <mechanicalReducction>1</mechanicalReducction>
+      </actuator>
+    </transmission>
+  </macro>
+  <wheel_trans prefix_name="left_front" />
+  <wheel_trans prefix_name="right_front" />
+  <wheel_trans prefix_name="left_rear" />
+  <wheel_trans prefix_name="right_rear" />
   <!-- Add Gazebo meterials tag -->
   <gazebo reference="libro_chassis_link">
@@ -17,4 +33,7 @@
       <material>Gazebo/FlatBlack</material>
  </gazebo>
+ <gazebo reference="ydlidar_link">
+      <material> Gazebo/Grey </material>
+ </gazebo>
   <!-- Add Gazebo ros control tag -->
   <gazebo>

File: libro_model/urdf/libro_model.urdf.xacro (robot description, xacro)
@@ -143,20 +143,57 @@
     <!-- <limit lower="-180" upper="180" effort="0" velocity="0" /> -->
   </joint>
-  <!-- Add transmission to each wheel joint -->
-  <macro name="wheel_trans" params="prefix_name">
-    <transmission name="${prefix_name}_wheel_transmission">
-      <type>transmission_interface/SimpleTransmission</type>
-      <joint name="${prefix_name}_wheel_joint">
-        <hardwareInterface>hardware_interface/VelocityJointInterface</hardwareInterface>
-      </joint>
-      <actuator name="${prefix_name}_wheel_motor">
-        <mechanicalReducction>1</mechanicalReducction>
-      </actuator>
-    </transmission>
-  </macro>
-  <wheel_trans prefix_name="left_front" />
-  <wheel_trans prefix_name="right_front" />
-  <wheel_trans prefix_name="left_rear" />
-  <wheel_trans prefix_name="right_rear" />
+    <link
+    name="ydlidar_link">
+    <inertial>
+      <origin
+        xyz="0.080408 0.0011599 0.020124"
+        rpy="0 0 0" />
+      <mass
+        value="0.05739" />
+      <inertia
+        ixx="1.3925E-05"
+        ixy="9.9078E-07"
+        ixz="-1.1243E-06"
+        iyy="3.4503E-05"
+        iyz="-1.2775E-07"
+        izz="4.723E-05" />
+    </inertial>
+    <visual>
+      <origin
+        xyz="0 0 0"
+        rpy="0 0 0" />
+      <geometry>
+        <mesh
+          filename="package://libro_model/meshes/ydlidar_link.STL" />
+      </geometry>
+      <material
+        name="">
+        <color
+          rgba="0.77255 0.75294 0.73333 1" />
+      </material>
+    </visual>
+    <collision>
+      <origin
+        xyz="0 0 0"
+        rpy="0 0 0" />
+      <geometry>
+        <mesh
+          filename="package://libro_model/meshes/ydlidar_link.STL" />
+      </geometry>
+    </collision>
+  </link>
+  <joint
+    name="ydlidar_joint"
+    type="fixed">
+    <origin
+      xyz="0 0 0"
+      rpy="0 0 0" />
+    <parent
+      link="libro_chassis_link" />
+    <child
+      link="ydlidar_link" />
+    <axis
+      xyz="0 0 0" />
+  </joint>
   <!-- base_link -->
   <link name="base_link"/>

Commit message: 添加了激光雷达插件

File: libro_model/urdf/gazebo_conf.xacro (robot description, xacro)
@@ -44,3 +44,35 @@
     </plugin>
   </gazebo>
+  <!-- Add YDLidar plugin -->
+  <gazebo reference="ydlidar_link">
+    <sensor type="ray" name="ydlidar_sensor">
+      <pose>0 0 0 0 0 0</pose>
+      <visualize>false</visualize>
+      <update_rate>40</update_rate>
+      <ray>
+        <scan>
+          <horizontal>
+            <samples>720</samples>
+            <resolution>1</resolution>
+            <min_angle>-1.570796</min_angle>
+            <max_angle>1.570796</max_angle>
+          </horizontal>
+        </scan>
+        <range>
+          <min>0.10</min>
+          <max>8.0</max>
+          <resolution>0.01</resolution>
+        </range>
+        <noise>
+          <type>gaussian</type>
+          <mean>0.0</mean>
+          <stddev>0.01</stddev>
+        </noise>
+      </ray>
+      <plugin name="gazebo_ros_ydlidar_controller" filename="libgazebo_ros_laser.so">
+        <topicName>/laser/scan</topicName>
+        <frameName>libro_chassis_link</frameName>
+      </plugin>
+    </sensor>
+  </gazebo>
  </robot>

File: libro_model/urdf/libro_model.urdf.xacro (robot description, xacro)
@@ -143,19 +143,19 @@
     <!-- <limit lower="-180" upper="180" effort="0" velocity="0" /> -->
   </joint>
-    <link
+  <link
     name="ydlidar_link">
     <inertial>
       <origin
-        xyz="0.080408 0.0011599 0.020124"
+        xyz="0.0231720323566563 0.00112954738407898 -0.045776403536883"
         rpy="0 0 0" />
       <mass
-        value="0.05739" />
+        value="0.0573896608078332" />
       <inertia
-        ixx="1.3925E-05"
-        ixy="9.9078E-07"
-        ixz="-1.1243E-06"
-        iyy="3.4503E-05"
-        iyz="-1.2775E-07"
-        izz="4.723E-05" />
+        ixx="1.39246903875836E-05"
+        ixy="9.90784550405998E-07"
+        ixz="-1.12428911988727E-06"
+        iyy="3.45029950880899E-05"
+        iyz="-1.27754764540977E-07"
+        izz="4.72303912642056E-05" />
     </inertial>
     <visual>
@@ -170,5 +170,5 @@
         name="">
         <color
-          rgba="0.77255 0.75294 0.73333 1" />
+          rgba="0.772549019607843 0.752941176470588 0.733333333333333 1" />
       </material>
     </visual>
@@ -185,4 +185,57 @@
   <joint
     name="ydlidar_joint"
+    type="fixed">
+    <origin
+      xyz="0.056136 -0.00016187 0.0859"
+      rpy="0 0 0" />
+    <parent
+      link="libro_chassis_link" />
+    <child
+      link="ydlidar_link" />
+    <axis
+      xyz="0 0 0" />
+  </joint>
+  <link
+    name="lidar_underframe_link">
+    <inertial>
+      <origin
+        xyz="0.0713736461903973 -9.66678635817838E-05 0.01"
+        rpy="0 0 0" />
+      <mass
+        value="0.119982831853072" />
+      <inertia
+        ixx="3.99842050248324E-05"
+        ixy="8.82530750051684E-21"
+        ixz="-7.14343913461121E-22"
+        iyy="0.000103956889382291"
+        iyz="5.54441914502247E-22"
+        izz="0.000135942238950252" />
+    </inertial>
+    <visual>
+      <origin
+        xyz="0 0 0"
+        rpy="0 0 0" />
+      <geometry>
+        <mesh
+          filename="package://libro_model/meshes/lidar_underframe_link.STL" />
+      </geometry>
+      <material
+        name="">
+        <color
+          rgba="1 1 1 1" />
+      </material>
+    </visual>
+    <collision>
+      <origin
+        xyz="0 0 0"
+        rpy="0 0 0" />
+      <geometry>
+        <mesh
+          filename="package://libro_model/meshes/lidar_underframe_link.STL" />
+      </geometry>
+    </collision>
+  </link>
+  <joint
+    name="lidar_underframe_joint"
     type="fixed">
     <origin
@@ -192,5 +245,5 @@
       link="libro_chassis_link" />
     <child
-      link="ydlidar_link" />
+      link="lidar_underframe_link" />
     <axis
       xyz="0 0 0" />

Commit message: 新增gmapping建图测试部分

File: libro_model/urdf/gazebo_conf.xacro (robot description, xacro)
@@ -22,18 +22,18 @@
   </gazebo>
   <gazebo reference="left_front_wheel_link">
-      <material>Gazebo/FlatBlack</material>
- </gazebo>
- <gazebo reference="right_front_wheel_link">
-      <material>Gazebo/FlatBlack</material>
- </gazebo>
- <gazebo reference="left_rear_wheel_link">
-      <material>Gazebo/FlatBlack</material>
- </gazebo>
- <gazebo reference="right_rear_wheel_link">
-      <material>Gazebo/FlatBlack</material>
- </gazebo>
- <gazebo reference="ydlidar_link">
-      <material> Gazebo/Grey </material>
- </gazebo>
+    <material>Gazebo/FlatBlack</material>
+  </gazebo>
+  <gazebo reference="right_front_wheel_link">
+    <material>Gazebo/FlatBlack</material>
+  </gazebo>
+  <gazebo reference="left_rear_wheel_link">
+    <material>Gazebo/FlatBlack</material>
+  </gazebo>
+  <gazebo reference="right_rear_wheel_link">
+    <material>Gazebo/FlatBlack</material>
+  </gazebo>
+  <gazebo reference="ydlidar_link">
+    <material> Gazebo/Grey </material>
+  </gazebo>
   <!-- Add Gazebo ros control tag -->
   <gazebo>
@@ -53,12 +53,12 @@
         <scan>
           <horizontal>
-            <samples>720</samples>
-            <resolution>1</resolution>
-            <min_angle>-1.570796</min_angle>
-            <max_angle>1.570796</max_angle>
+            <samples>700</samples>
+            <resolution>0.84</resolution>
+            <min_angle>-3.1415926</min_angle>
+            <max_angle>3.1415926</max_angle>
           </horizontal>
         </scan>
         <range>
-          <min>0.10</min>
+          <min>0.1</min>
           <max>8.0</max>
           <resolution>0.01</resolution>
@@ -76,3 +76,3 @@
     </sensor>
   </gazebo>
- </robot>
+</robot>

Commit message: 更改了驱动方式

File: libro_model/urdf/gazebo_conf.xacro (robot description, xacro)
@@ -22,13 +22,21 @@
   </gazebo>
   <gazebo reference="left_front_wheel_link">
+    <mu1>0.2</mu1>
+    <mu2>0.2</mu2>
     <material>Gazebo/FlatBlack</material>
   </gazebo>
   <gazebo reference="right_front_wheel_link">
+    <mu1>0.2</mu1>
+    <mu2>0.2</mu2>
     <material>Gazebo/FlatBlack</material>
   </gazebo>
   <gazebo reference="left_rear_wheel_link">
+    <mu1>0.2</mu1>
+    <mu2>0.2</mu2>
     <material>Gazebo/FlatBlack</material>
   </gazebo>
   <gazebo reference="right_rear_wheel_link">
+    <mu1>0.2</mu1>
+    <mu2>0.2</mu2>
     <material>Gazebo/FlatBlack</material>
   </gazebo>
@@ -44,4 +52,23 @@
     </plugin>
   </gazebo>
+  <gazebo>
+    <plugin name="skid_steer_drive_controller" filename="libgazebo_ros_skid_steer_drive.so">
+      <alwaysOn>true</alwaysOn>
+      <updateRate>100.0</updateRate>
+      <robotNamespace>/</robotNamespace>
+      <leftFrontJoint>left_front_wheel_joint</leftFrontJoint>
+      <rightFrontJoint>right_front_wheel_joint</rightFrontJoint>
+      <leftRearJoint>left_rear_wheel_joint</leftRearJoint>
+      <rightRearJoint>right_rear_wheel_joint</rightRearJoint>
+      <wheelSeparation>0.12</wheelSeparation>
+      <wheelDiameter>0.065</wheelDiameter>
+      <torque>2.6</torque>
+      <commandTopic>cmd_vel</commandTopic>
+      <odometryTopic>odom</odometryTopic>
+      <odometryFrame>odom</odometryFrame>
+      <robotBaseFrame>base_link</robotBaseFrame>
+      <broadcastTF>1</broadcastTF>
+    </plugin>
+  </gazebo>
   <!-- Add YDLidar plugin -->
   <gazebo reference="ydlidar_link">
@@ -49,5 +76,5 @@
       <pose>0 0 0 0 0 0</pose>
       <visualize>false</visualize>
-      <update_rate>60</update_rate>
+      <update_rate>40</update_rate>
       <ray>
         <scan>

File: libro_model/urdf/libro_model.urdf.xacro (robot description, xacro)
@@ -5,4 +5,26 @@
 <robot name="libro_model"
   xmlns:xacro="http://ros.org/wiki/xacro">
+  <link name="base_footprint">
+        <visual>
+            <geometry>
+                    <box size="0.001 0.001 0.001"/>
+                </geometry>
+            <origin rpy="0 0 0" xyz="0 0 0"/>
+        </visual>
+       <inertial>
+                       <mass value="0.0001" />
+                       <inertia ixx="1.0" ixy="0.0" ixz="0.0"
+                                iyy="1.0" iyz="0.0"
+                                izz="1.0" />
+               </inertial>
+    </link>
+    <gazebo reference="base_footprint">
+        <turnGravityOff>false</turnGravityOff>
+    </gazebo>
+    <joint name="base_footprint_joint" type="fixed">
+        <origin xyz="0 0 0" />
+        <parent link="base_footprint" />
+        <child link="base_link" />
+    </joint>
   <link name="libro_chassis_link">
     <inertial>
