Commit message: 修正了跳跳车的bug

File: libro_model/urdf/gazebo_conf.xacro (robot description, xacro)
@@ -18,4 +18,7 @@
   <wheel_trans prefix_name="right_rear" />
   <!-- Add Gazebo meterials tag -->
+  <gazebo reference="base_footprint">
+    <turnGravityOff>false</turnGravityOff>
+  </gazebo>
   <gazebo reference="libro_chassis_link">
     <material>Gazebo/White</material>
@@ -44,12 +47,4 @@
     <material> Gazebo/Grey </material>
   </gazebo>
-  <!-- Add Gazebo ros control tag -->
-  <gazebo>
-    <plugin name="gazebo_ros_control" filename="libgazebo_ros_control.so">
-      <robotNamespace>/</robotNamespace>
-      <robotSimType>gazebo_ros_control/DefaultRobotHWSim</robotSimType>
-      <legacyModeNS>true</legacyModeNS>
-    </plugin>
-  </gazebo>
   <gazebo>
     <plugin name="skid_steer_drive_controller" filename="libgazebo_ros_skid_steer_drive.so">
@@ -63,10 +58,13 @@
       <wheelSeparation>0.12</wheelSeparation>
       <wheelDiameter>0.065</wheelDiameter>
-      <torque>2.6</torque>
+      <torque>2</torque>
       <commandTopic>cmd_vel</commandTopic>
       <odometryTopic>odom</odometryTopic>
       <odometryFrame>odom</odometryFrame>
-      <robotBaseFrame>base_link</robotBaseFrame>
+      <robotBaseFrame>base_footprint</robotBaseFrame>
       <broadcastTF>1</broadcastTF>
+      <covariance_x>0.0001</covariance_x>
+      <covariance_y>0.0001</covariance_y>
+      <covariance_yaw>0.01</covariance_yaw>
     </plugin>
   </gazebo>
@@ -99,5 +97,5 @@
       <plugin name="gazebo_ros_ydlidar_controller" filename="libgazebo_ros_laser.so">
         <topicName>/laser/scan</topicName>
-        <frameName>base_link</frameName>
+        <frameName>ydlidar_link</frameName>
       </plugin>
     </sensor>

File: libro_model/urdf/libro_model.urdf.xacro (robot description, xacro)
@@ -5,271 +5,10 @@
 <robot name="libro_model"
   xmlns:xacro="http://ros.org/wiki/xacro">
-  <link name="base_footprint">
-        <visual>
-            <geometry>
-                    <box size="0.001 0.001 0.001"/>
-                </geometry>
-            <origin rpy="0 0 0" xyz="0 0 0"/>
-        </visual>
-       <inertial>
-                       <mass value="0.0001" />
-                       <inertia ixx="1.0" ixy="0.0" ixz="0.0"
-                                iyy="1.0" iyz="0.0"
-                                izz="1.0" />
-               </inertial>
-    </link>
-    <gazebo reference="base_footprint">
-        <turnGravityOff>false</turnGravityOff>
-    </gazebo>
-    <joint name="base_footprint_joint" type="fixed">
-        <origin xyz="0 0 0" />
-        <parent link="base_footprint" />
-        <child link="base_link" />
-    </joint>
-  <link name="libro_chassis_link">
-    <inertial>
-      <origin xyz="5.68208583529243E-05 -1.08190137895018E-05 -0.0191328128743083" rpy="0 0 0" />
-      <mass value="0.315959634168836" />
-      <inertia ixx="0.000237187119369315" ixy="1.02623528819012E-07" ixz="-5.76554239644837E-20" iyy="0.000984715228403803" iyz="3.46081831405105E-20" izz="0.00120943275258583" />
-    </inertial>
-    <visual>
-      <origin xyz="0 0 0" rpy="0 0 0" />
-      <geometry>
-        <mesh filename="package://libro_model/meshes/base_link.STL" />
-      </geometry>
-      <material name="">
-        <color rgba="1 1 1 1" />
-      </material>
-    </visual>
-    <collision>
-      <origin xyz="0 0 0" rpy="0 0 0" />
-      <geometry>
-        <mesh filename="package://libro_model/meshes/base_link.STL" />
-      </geometry>
-    </collision>
-  </link>
-  <link name="right_front_wheel_link">
-    <inertial>
-      <origin xyz="1.38777878078145E-17 0.000536215321318312 3.46944695195361E-18" rpy="0 0 0" />
-      <mass value="0.0420890500835263" />
-      <inertia ixx="1.69788467809493E-05" ixy="-1.07143056154772E-22" ixz="3.59209508752315E-22" iyy="2.82266239844783E-05" iyz="2.23488333501653E-21" izz="1.69803313609295E-05" />
-    </inertial>
-    <visual>
-      <origin xyz="0 0 0" rpy="0 0 0" />
-      <geometry>
-        <mesh filename="package://libro_model/meshes/right_front_wheel_link.STL" />
-      </geometry>
-      <material name="">
-        <color rgba="0.298039215686275 0.298039215686275 0.298039215686275 1" />
-      </material>
-    </visual>
-    <collision>
-      <origin xyz="0 0 0" rpy="0 0 0" />
-      <geometry>
-        <mesh filename="package://libro_model/meshes/right_front_wheel_link.STL" />
-      </geometry>
-    </collision>
-  </link>
-  <joint name="right_front_wheel_joint" type="continuous">
-    <origin xyz="0.057307 -0.064491 -0.02175" rpy="0 0 0" />
-    <parent link="libro_chassis_link" />
-    <child link="right_front_wheel_link" />
-    <axis xyz="0 1 0" />
-    <!-- <limit lower="-180" upper="180" effort="0" velocity="0" /> -->
-  </joint>
-  <link name="right_rear_wheel_link">
-    <inertial>
-      <origin xyz="1.38777878078145E-17 0.000536215321318284 6.93889390390723E-18" rpy="0 0 0" />
-      <mass value="0.0420890500835264" />
-      <inertia ixx="1.69788467809493E-05" ixy="1.57919887602203E-21" ixz="-3.34928854973574E-22" iyy="2.82266239844783E-05" iyz="3.29921671584904E-22" izz="1.69803313609295E-05" />
-    </inertial>
-    <visual>
-      <origin xyz="0 0 0" rpy="0 0 0" />
-      <geometry>
-        <mesh filename="package://libro_model/meshes/right_rear_wheel_link.STL" />
-      </geometry>
-      <material name="">
-        <color rgba="0.298039215686275 0.298039215686275 0.298039215686275 1" />
-      </material>
-    </visual>
-    <collision>
-      <origin xyz="0 0 0" rpy="0 0 0" />
-      <geometry>
-        <mesh filename="package://libro_model/meshes/right_rear_wheel_link.STL" />
-      </geometry>
-    </collision>
-  </link>
-  <joint name="right_rear_wheel_joint" type="continuous">
-    <origin xyz="-0.057693 -0.064454 -0.02175" rpy="0 0 0" />
-    <parent link="libro_chassis_link" />
-    <child link="right_rear_wheel_link" />
-    <axis xyz="0 1 0" />
-    <!-- <limit lower="-180" upper="180" effort="0" velocity="0" /> -->
-  </joint>
-  <link name="left_front_wheel_link">
-    <inertial>
-      <origin xyz="-6.93889390390723E-18 -0.000536215321318298 0" rpy="0 0 0" />
-      <mass value="0.0420890500835263" />
-      <inertia ixx="1.69788467809493E-05" ixy="1.20055989289706E-21" ixz="-3.34719610585716E-22" iyy="2.82266239844783E-05" iyz="-1.25731607683899E-21" izz="1.69803313609295E-05" />
-    </inertial>
-    <visual>
-      <origin xyz="0 0 0" rpy="0 0 0" />
-      <geometry>
-        <mesh filename="package://libro_model/meshes/left_front_wheel_link.STL" />
-      </geometry>
-      <material name="">
-        <color rgba="0.298039215686275 0.298039215686275 0.298039215686275 1" />
-      </material>
-    </visual>
-    <collision>
-      <origin xyz="0 0 0" rpy="0 0 0" />
-      <geometry>
-        <mesh filename="package://libro_model/meshes/left_front_wheel_link.STL" />
-      </geometry>
-    </collision>
-  </link>
-  <joint name="left_front_wheel_joint" type="continuous">
-    <origin xyz="0.057307 0.064455 -0.02175" rpy="0 0 0" />
-    <parent link="libro_chassis_link" />
-    <child link="left_front_wheel_link" />
-    <axis xyz="0 1 0" />
-    <!-- <limit lower="-180" upper="180" effort="0" velocity="0" /> -->
-  </joint>
-  <link name="left_rear_wheel_link">
-    <inertial>
-      <origin xyz="4.16333634234434E-17 -0.000536215321318353 -3.46944695195361E-16" rpy="0 0 0" />
-      <mass value="0.0420890500835263" />
-      <inertia ixx="1.69788496293646E-05" ixy="-1.18719665581258E-21" ixz="6.49660441239981E-11" iyy="2.82266239844783E-05" iyz="1.01365580326182E-21" izz="1.69803285125142E-05" />
-    </inertial>
-    <visual>
-      <origin xyz="0 0 0" rpy="0 0 0" />
-      <geometry>
-        <mesh filename="package://libro_model/meshes/left_rear_wheel_link.STL" />
-      </geometry>
-      <material name="">
-        <color rgba="0.298039215686275 0.298039215686275 0.298039215686275 1" />
-      </material>
-    </visual>
-    <collision>
-      <origin xyz="0 0 0" rpy="0 0 0" />
-      <geometry>
-        <mesh filename="package://libro_model/meshes/left_rear_wheel_link.STL" />
-      </geometry>
-    </collision>
-  </link>
-  <joint name="left_rear_wheel_joint" type="continuous">
-    <origin xyz="-0.057693 0.064369 -0.02175" rpy="0 0 0" />
-    <parent link="libro_chassis_link" />
-    <child link="left_rear_wheel_link" />
-    <axis xyz="0 1 0" />
-    <!-- <limit lower="-180" upper="180" effort="0" velocity="0" /> -->
-  </joint>
-  <link
-    name="ydlidar_link">
-    <inertial>
-      <origin
-        xyz="0.0231720323566563 0.00112954738407898 -0.045776403536883"
-        rpy="0 0 0" />
-      <mass
-        value="0.0573896608078332" />
-      <inertia
-        ixx="1.39246903875836E-05"
-        ixy="9.90784550405998E-07"
-        ixz="-1.12428911988727E-06"
-        iyy="3.45029950880899E-05"
-        iyz="-1.27754764540977E-07"
-        izz="4.72303912642056E-05" />
-    </inertial>
-    <visual>
-      <origin
-        xyz="0 0 0"
-        rpy="0 0 0" />
-      <geometry>
-        <mesh
-          filename="package://libro_model/meshes/ydlidar_link.STL" />
-      </geometry>
-      <material
-        name="">
-        <color
-          rgba="0.772549019607843 0.752941176470588 0.733333333333333 1" />
-      </material>
-    </visual>
-    <collision>
-      <origin
-        xyz="0 0 0"
-        rpy="0 0 0" />
-      <geometry>
-        <mesh
-          filename="package://libro_model/meshes/ydlidar_link.STL" />
-      </geometry>
-    </collision>
-  </link>
-  <joint
-    name="ydlidar_joint"
-    type="fixed">
-    <origin
-      xyz="0.056136 -0.00016187 0.0859"
-      rpy="0 0 0" />
-    <parent
-      link="libro_chassis_link" />
-    <child
-      link="ydlidar_link" />
-    <axis
-      xyz="0 0 0" />
-  </joint>
-  <link
-    name="lidar_underframe_link">
-    <inertial>
-      <origin
-        xyz="0.0713736461903973 -9.66678635817838E-05 0.01"
-        rpy="0 0 0" />
-      <mass
-        value="0.119982831853072" />
-      <inertia
-        ixx="3.99842050248324E-05"
-        ixy="8.82530750051684E-21"
-        ixz="-7.14343913461121E-22"
-        iyy="0.000103956889382291"
-        iyz="5.54441914502247E-22"
-        izz="0.000135942238950252" />
-    </inertial>
-    <visual>
-      <origin
-        xyz="0 0 0"
-        rpy="0 0 0" />
-      <geometry>
-        <mesh
-          filename="package://libro_model/meshes/lidar_underframe_link.STL" />
-      </geometry>
-      <material
-        name="">
-        <color
-          rgba="1 1 1 1" />
-      </material>
-    </visual>
-    <collision>
-      <origin
-        xyz="0 0 0"
-        rpy="0 0 0" />
-      <geometry>
-        <mesh
-          filename="package://libro_model/meshes/lidar_underframe_link.STL" />
-      </geometry>
-    </collision>
-  </link>
-  <joint
-    name="lidar_underframe_joint"
-    type="fixed">
-    <origin
-      xyz="0 0 0"
-      rpy="0 0 0" />
-    <parent
-      link="libro_chassis_link" />
-    <child
-      link="lidar_underframe_link" />
-    <axis
-      xyz="0 0 0" />
-  </joint>
-  <!-- base_link -->
+  <link name="base_footprint" />
+  <joint name="base_footprint_joint" type="fixed">
+    <origin xyz="0 0 0.04" rpy="0.0 0.0 0.0"/>
+    <parent link="base_footprint" />
+    <child link="base_link" />
+  </joint>
   <link name="base_link"/>
   <joint name="base_joint" type="fixed">
@@ -278,3 +17,197 @@
     <child link="libro_chassis_link"/>
   </joint>
+  <link name="libro_chassis_link">
+    <inertial>
+      <origin xyz="5.68208583529243E-05 -1.08190137895018E-05 -0.0191328128743083" rpy="0 0 0" />
+      <mass value="0.315959634168836" />
+      <inertia ixx="0.000237187119369315" ixy="1.02623528819012E-07" ixz="-5.76554239644837E-20" iyy="0.000984715228403803" iyz="3.46081831405105E-20" izz="0.00120943275258583" />
+    </inertial>
+    <visual>
+      <origin xyz="0 0 0" rpy="0 0 0" />
+      <geometry>
+        <mesh filename="package://libro_model/meshes/base_link.STL" />
+      </geometry>
+      <material name="">
+        <color rgba="1 1 1 1" />
+      </material>
+    </visual>
+    <collision>
+      <origin xyz="0 0 0" rpy="0 0 0" />
+      <geometry>
+        <mesh filename="package://libro_model/meshes/base_link.STL" />
+      </geometry>
+    </collision>
+  </link>
+  <link name="right_front_wheel_link">
+    <inertial>
+      <origin xyz="1.38777878078145E-17 0.000536215321318312 3.46944695195361E-18" rpy="0 0 0" />
+      <mass value="0.0420890500835263" />
+      <inertia ixx="1.69788467809493E-05" ixy="-1.07143056154772E-22" ixz="3.59209508752315E-22" iyy="2.82266239844783E-05" iyz="2.23488333501653E-21" izz="1.69803313609295E-05" />
+    </inertial>
+    <visual>
+      <origin xyz="0 0 0" rpy="0 0 0" />
+      <geometry>
+        <mesh filename="package://libro_model/meshes/right_front_wheel_link.STL" />
+      </geometry>
+      <material name="">
+        <color rgba="0.298039215686275 0.298039215686275 0.298039215686275 1" />
+      </material>
+    </visual>
+    <collision>
+      <origin xyz="0 0 0" rpy="0 0 0" />
+      <geometry>
+        <mesh filename="package://libro_model/meshes/right_front_wheel_link.STL" />
+      </geometry>
+    </collision>
+  </link>
+  <joint name="right_front_wheel_joint" type="continuous">
+    <origin xyz="0.057307 -0.064491 -0.02175" rpy="0 0 0" />
+    <parent link="libro_chassis_link" />
+    <child link="right_front_wheel_link" />
+    <axis xyz="0 1 0" />
+    <!-- <limit lower="-180" upper="180" effort="0" velocity="0" /> -->
+  </joint>
+  <link name="right_rear_wheel_link">
+    <inertial>
+      <origin xyz="1.38777878078145E-17 0.000536215321318284 6.93889390390723E-18" rpy="0 0 0" />
+      <mass value="0.0420890500835264" />
+      <inertia ixx="1.69788467809493E-05" ixy="1.57919887602203E-21" ixz="-3.34928854973574E-22" iyy="2.82266239844783E-05" iyz="3.29921671584904E-22" izz="1.69803313609295E-05" />
+    </inertial>
+    <visual>
+      <origin xyz="0 0 0" rpy="0 0 0" />
+      <geometry>
+        <mesh filename="package://libro_model/meshes/right_rear_wheel_link.STL" />
+      </geometry>
+      <material name="">
+        <color rgba="0.298039215686275 0.298039215686275 0.298039215686275 1" />
+      </material>
+    </visual>
+    <collision>
+      <origin xyz="0 0 0" rpy="0 0 0" />
+      <geometry>
+        <mesh filename="package://libro_model/meshes/right_rear_wheel_link.STL" />
+      </geometry>
+    </collision>
+  </link>
+  <joint name="right_rear_wheel_joint" type="continuous">
+    <origin xyz="-0.057693 -0.064454 -0.02175" rpy="0 0 0" />
+    <parent link="libro_chassis_link" />
+    <child link="right_rear_wheel_link" />
+    <axis xyz="0 1 0" />
+    <!-- <limit lower="-180" upper="180" effort="0" velocity="0" /> -->
+  </joint>
+  <link name="left_front_wheel_link">
+    <inertial>
+      <origin xyz="-6.93889390390723E-18 -0.000536215321318298 0" rpy="0 0 0" />
+      <mass value="0.0420890500835263" />
+      <inertia ixx="1.69788467809493E-05" ixy="1.20055989289706E-21" ixz="-3.34719610585716E-22" iyy="2.82266239844783E-05" iyz="-1.25731607683899E-21" izz="1.69803313609295E-05" />
+    </inertial>
+    <visual>
+      <origin xyz="0 0 0" rpy="0 0 0" />
+      <geometry>
+        <mesh filename="package://libro_model/meshes/left_front_wheel_link.STL" />
+      </geometry>
+      <material name="">
+        <color rgba="0.298039215686275 0.298039215686275 0.298039215686275 1" />
+      </material>
+    </visual>
+    <collision>
+      <origin xyz="0 0 0" rpy="0 0 0" />
+      <geometry>
+        <mesh filename="package://libro_model/meshes/left_front_wheel_link.STL" />
+      </geometry>
+    </collision>
+  </link>
+  <joint name="left_front_wheel_joint" type="continuous">
+    <origin xyz="0.057307 0.064455 -0.02175" rpy="0 0 0" />
+    <parent link="libro_chassis_link" />
+    <child link="left_front_wheel_link" />
+    <axis xyz="0 1 0" />
+    <!-- <limit lower="-180" upper="180" effort="0" velocity="0" /> -->
+  </joint>
+  <link name="left_rear_wheel_link">
+    <inertial>
+      <origin xyz="4.16333634234434E-17 -0.000536215321318353 -3.46944695195361E-16" rpy="0 0 0" />
+      <mass value="0.0420890500835263" />
+      <inertia ixx="1.69788496293646E-05" ixy="-1.18719665581258E-21" ixz="6.49660441239981E-11" iyy="2.82266239844783E-05" iyz="1.01365580326182E-21" izz="1.69803285125142E-05" />
+    </inertial>
+    <visual>
+      <origin xyz="0 0 0" rpy="0 0 0" />
+      <geometry>
+        <mesh filename="package://libro_model/meshes/left_rear_wheel_link.STL" />
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