Commit message: Merge branch 'dev' of github.com:df-club/libro into dev

File: libro_model/urdf/libro_model.urdf.xacro (robot description, xacro)
@@ -7,5 +7,5 @@
   <link name="base_footprint" />
   <joint name="base_footprint_joint" type="fixed">
-    <origin xyz="0 0 0.04" rpy="0.0 0.0 0.0"/>
+    <origin xyz="0 0 0.055" rpy="0.0 0.0 0.0"/>
     <parent link="base_footprint" />
     <child link="base_link" />

Commit message: 整理项目的文件夹结构

File: libro_model/urdf/libro_model.urdf.xacro (robot description, xacro)
@@ -26,5 +26,5 @@
       <origin xyz="0 0 0" rpy="0 0 0" />
       <geometry>
-        <mesh filename="package://libro_model/meshes/base_link.STL" />
+        <mesh filename="package://libro_model/urdf/meshes/base_link.STL" />
       </geometry>
       <material name="">
@@ -35,5 +35,5 @@
       <origin xyz="0 0 0" rpy="0 0 0" />
       <geometry>
-        <mesh filename="package://libro_model/meshes/base_link.STL" />
+        <mesh filename="package://libro_model/urdf/meshes/base_link.STL" />
       </geometry>
     </collision>
@@ -48,14 +48,14 @@
       <origin xyz="0 0 0" rpy="0 0 0" />
       <geometry>
-        <mesh filename="package://libro_model/meshes/right_front_wheel_link.STL" />
-      </geometry>
-      <material name="">
-        <color rgba="0.298039215686275 0.298039215686275 0.298039215686275 1" />
-      </material>
-    </visual>
-    <collision>
-      <origin xyz="0 0 0" rpy="0 0 0" />
-      <geometry>
-        <mesh filename="package://libro_model/meshes/right_front_wheel_link.STL" />
+        <mesh filename="package://libro_model/urdf/meshes/right_front_wheel_link.STL" />
+      </geometry>
+      <material name="">
+        <color rgba="0.298039215686275 0.298039215686275 0.298039215686275 1" />
+      </material>
+    </visual>
+    <collision>
+      <origin xyz="0 0 0" rpy="0 0 0" />
+      <geometry>
+        <mesh filename="package://libro_model/urdf/meshes/right_front_wheel_link.STL" />
       </geometry>
     </collision>
@@ -77,14 +77,14 @@
       <origin xyz="0 0 0" rpy="0 0 0" />
       <geometry>
-        <mesh filename="package://libro_model/meshes/right_rear_wheel_link.STL" />
-      </geometry>
-      <material name="">
-        <color rgba="0.298039215686275 0.298039215686275 0.298039215686275 1" />
-      </material>
-    </visual>
-    <collision>
-      <origin xyz="0 0 0" rpy="0 0 0" />
-      <geometry>
-        <mesh filename="package://libro_model/meshes/right_rear_wheel_link.STL" />
+        <mesh filename="package://libro_model/urdf/meshes/right_rear_wheel_link.STL" />
+      </geometry>
+      <material name="">
+        <color rgba="0.298039215686275 0.298039215686275 0.298039215686275 1" />
+      </material>
+    </visual>
+    <collision>
+      <origin xyz="0 0 0" rpy="0 0 0" />
+      <geometry>
+        <mesh filename="package://libro_model/urdf/meshes/right_rear_wheel_link.STL" />
       </geometry>
     </collision>
@@ -106,14 +106,14 @@
       <origin xyz="0 0 0" rpy="0 0 0" />
       <geometry>
-        <mesh filename="package://libro_model/meshes/left_front_wheel_link.STL" />
-      </geometry>
-      <material name="">
-        <color rgba="0.298039215686275 0.298039215686275 0.298039215686275 1" />
-      </material>
-    </visual>
-    <collision>
-      <origin xyz="0 0 0" rpy="0 0 0" />
-      <geometry>
-        <mesh filename="package://libro_model/meshes/left_front_wheel_link.STL" />
+        <mesh filename="package://libro_model/urdf/meshes/left_front_wheel_link.STL" />
+      </geometry>
+      <material name="">
+        <color rgba="0.298039215686275 0.298039215686275 0.298039215686275 1" />
+      </material>
+    </visual>
+    <collision>
+      <origin xyz="0 0 0" rpy="0 0 0" />
+      <geometry>
+        <mesh filename="package://libro_model/urdf/meshes/left_front_wheel_link.STL" />
       </geometry>
     </collision>
@@ -135,14 +135,14 @@
       <origin xyz="0 0 0" rpy="0 0 0" />
       <geometry>
-        <mesh filename="package://libro_model/meshes/left_rear_wheel_link.STL" />
-      </geometry>
-      <material name="">
-        <color rgba="0.298039215686275 0.298039215686275 0.298039215686275 1" />
-      </material>
-    </visual>
-    <collision>
-      <origin xyz="0 0 0" rpy="0 0 0" />
-      <geometry>
-        <mesh filename="package://libro_model/meshes/left_rear_wheel_link.STL" />
+        <mesh filename="package://libro_model/urdf/meshes/left_rear_wheel_link.STL" />
+      </geometry>
+      <material name="">
+        <color rgba="0.298039215686275 0.298039215686275 0.298039215686275 1" />
+      </material>
+    </visual>
+    <collision>
+      <origin xyz="0 0 0" rpy="0 0 0" />
+      <geometry>
+        <mesh filename="package://libro_model/urdf/meshes/left_rear_wheel_link.STL" />
       </geometry>
     </collision>
@@ -164,5 +164,5 @@
       <origin xyz="0 0 0" rpy="0 0 0" />
       <geometry>
-        <mesh filename="package://libro_model/meshes/ydlidar_link.STL" />
+        <mesh filename="package://libro_model/urdf/meshes/ydlidar_link.STL" />
       </geometry>
       <material name="">
@@ -173,5 +173,5 @@
       <origin xyz="0 0 0" rpy="0 0 0" />
       <geometry>
-        <mesh filename="package://libro_model/meshes/ydlidar_link.STL" />
+        <mesh filename="package://libro_model/urdf/meshes/ydlidar_link.STL" />
       </geometry>
     </collision>
@@ -192,5 +192,5 @@
       <origin xyz="0 0 0" rpy="0 0 0" />
       <geometry>
-        <mesh filename="package://libro_model/meshes/lidar_underframe_link.STL" />
+        <mesh filename="package://libro_model/urdf/meshes/lidar_underframe_link.STL" />
       </geometry>
       <material name="">
@@ -201,5 +201,5 @@
       <origin xyz="0 0 0" rpy="0 0 0" />
       <geometry>
-        <mesh filename="package://libro_model/meshes/lidar_underframe_link.STL" />
+        <mesh filename="package://libro_model/urdf/meshes/lidar_underframe_link.STL" />
       </geometry>
     </collision>

Commit message: 添加IMU惯性导航模块，使用imu和里程计混合的odom

File: libro_model/urdf/libro_model.urdf.xacro (robot description, xacro)
@@ -211,3 +211,25 @@
     <axis xyz="0 0 0" />
   </joint>
+  <link name="imu_link">
+    <inertial>
+      <mass value="0.01" />
+      <inertia ixx="1.0" ixy="0.0" ixz="0.0" iyy="1.0" iyz="0.0" izz="1.0" />
+    </inertial>
+    <visual>
+      <geometry>
+        <box size="0.01 0.01 0.01"/>
+      </geometry>
+    </visual>
+    <collision>
+      <geometry>
+        <box size="0.01 0.01 0.01"/>
+      </geometry>
+    </collision>
+  </link>
+  <joint name="imu_joint" type="fixed">
+    <origin xyz="0 0 0" rpy="0 0 0" />
+    <parent link="libro_chassis_link" />
+    <child link="imu_link" />
+    <axis xyz="0 0 0" />
+  </joint>
 </robot>

Commit message: 添加了摄像头模型

File: libro_model/urdf/libro_model.urdf.xacro (robot description, xacro)
@@ -211,25 +211,31 @@
     <axis xyz="0 0 0" />
   </joint>
-  <link name="imu_link">
-    <inertial>
-      <mass value="0.01" />
-      <inertia ixx="1.0" ixy="0.0" ixz="0.0" iyy="1.0" iyz="0.0" izz="1.0" />
-    </inertial>
-    <visual>
-      <geometry>
-        <box size="0.01 0.01 0.01"/>
-      </geometry>
-    </visual>
-    <collision>
-      <geometry>
-        <box size="0.01 0.01 0.01"/>
-      </geometry>
-    </collision>
-  </link>
-  <joint name="imu_joint" type="fixed">
-    <origin xyz="0 0 0" rpy="0 0 0" />
-    <parent link="libro_chassis_link" />
-    <child link="imu_link" />
-    <axis xyz="0 0 0" />
+  <link name="camera_link">
+    <inertial>
+      <origin xyz="-0.00303115254709119 9.98333360424652E-16 -5.12569483805715E-05"  rpy="0 0 0" />
+      <mass value="0.00145671307075292" />
+      <inertia  ixx="6.93646665527772E-08" ixy="3.04630454817989E-24" ixz="-1.09673943150479E-10"  iyy="3.98881873637141E-08"  iyz="-9.33337790838574E-24"  izz="3.98920145491929E-08" />
+    </inertial>
+    <visual>
+      <origin xyz="0 0 0"  rpy="0 0 0" />
+      <geometry>
+        <mesh filename="package://libro_model/urdf/meshes/camera_link.STL" />
+      </geometry>
+      <material  name="">
+        <color rgba="1 1 1 1" />
+      </material>
+    </visual>
+    <collision>
+      <origin xyz="0 0 0"  rpy="0 0 0" />
+      <geometry>
+        <mesh  filename="package://libro_model/urdf/meshes/camera_link.STL" />
+      </geometry>
+    </collision>
+  </link>
+  <joint name="camera_joint" type="fixed">
+    <origin  xyz="0.12531 -0.00043191 -0.023" rpy="0 0 0" />
+    <parent  link="libro_chassis_link" />
+    <child link="camera_link" />
+    <axis  xyz="0 1 0" />
   </joint>
 </robot>

Commit message: 重新添加了IMU模块

File: libro_model/urdf/libro_model.urdf.xacro (robot description, xacro)
@@ -213,29 +213,51 @@
   <link name="camera_link">
     <inertial>
-      <origin xyz="-0.00303115254709119 9.98333360424652E-16 -5.12569483805715E-05"  rpy="0 0 0" />
+      <origin xyz="-0.00303115254709119 9.98333360424652E-16 -5.12569483805715E-05" rpy="0 0 0" />
       <mass value="0.00145671307075292" />
-      <inertia  ixx="6.93646665527772E-08" ixy="3.04630454817989E-24" ixz="-1.09673943150479E-10"  iyy="3.98881873637141E-08"  iyz="-9.33337790838574E-24"  izz="3.98920145491929E-08" />
-    </inertial>
-    <visual>
-      <origin xyz="0 0 0"  rpy="0 0 0" />
+      <inertia ixx="6.93646665527772E-08" ixy="3.04630454817989E-24" ixz="-1.09673943150479E-10" iyy="3.98881873637141E-08" iyz="-9.33337790838574E-24" izz="3.98920145491929E-08" />
+    </inertial>
+    <visual>
+      <origin xyz="0 0 0" rpy="0 0 0" />
       <geometry>
         <mesh filename="package://libro_model/urdf/meshes/camera_link.STL" />
       </geometry>
-      <material  name="">
+      <material name="">
         <color rgba="1 1 1 1" />
       </material>
     </visual>
     <collision>
-      <origin xyz="0 0 0"  rpy="0 0 0" />
-      <geometry>
-        <mesh  filename="package://libro_model/urdf/meshes/camera_link.STL" />
+      <origin xyz="0 0 0" rpy="0 0 0" />
+      <geometry>
+        <mesh filename="package://libro_model/urdf/meshes/camera_link.STL" />
       </geometry>
     </collision>
   </link>
   <joint name="camera_joint" type="fixed">
-    <origin  xyz="0.12531 -0.00043191 -0.023" rpy="0 0 0" />
-    <parent  link="libro_chassis_link" />
+    <origin xyz="0.12531 -0.00043191 -0.023" rpy="0 0 0" />
+    <parent link="libro_chassis_link" />
     <child link="camera_link" />
-    <axis  xyz="0 1 0" />
+    <axis xyz="0 1 0" />
+  </joint>
+  <link name="imu_link">
+    <inertial>
+      <mass value="0.01" />
+      <inertia ixx="1.0" ixy="0.0" ixz="0.0" iyy="1.0" iyz="0.0" izz="1.0" />
+    </inertial>
+    <visual>
+      <geometry>
+        <box size="0.01 0.01 0.01"/>
+      </geometry>
+    </visual>
+    <collision>
+      <geometry>
+        <box size="0.01 0.01 0.01"/>
+      </geometry>
+    </collision>
+  </link>
+  <joint name="imu_joint" type="fixed">
+    <origin xyz="0 0 0" rpy="0 0 0" />
+    <parent link="libro_chassis_link" />
+    <child link="imu_link" />
+    <axis xyz="0 0 0" />
   </joint>
 </robot>

Commit message: 解决了速度变慢的问题

File: libro_model/urdf/libro_model.urdf.xacro (robot description, xacro)
@@ -240,8 +240,4 @@
   </joint>
   <link name="imu_link">
-    <inertial>
-      <mass value="0.01" />
-      <inertia ixx="1.0" ixy="0.0" ixz="0.0" iyy="1.0" iyz="0.0" izz="1.0" />
-    </inertial>
     <visual>
       <geometry>
@@ -249,12 +245,7 @@
       </geometry>
     </visual>
-    <collision>
-      <geometry>
-        <box size="0.01 0.01 0.01"/>
-      </geometry>
-    </collision>
   </link>
   <joint name="imu_joint" type="fixed">
-    <origin xyz="0 0 0" rpy="0 0 0" />
+    <origin xyz="0 0 0.01" rpy="0 0 0" />
     <parent link="libro_chassis_link" />
     <child link="imu_link" />

Commit message: 添加了imu和摄像头
Co-Authored-By: john1217 <13514609+john1217@users.noreply.github.com>
Co-Authored-By: Damongzx <77727892+Damongzx@users.noreply.github.com>

File: libro_model/urdf/libro_model.urdf.xacro (robot description, xacro)
@@ -26,5 +26,5 @@
       <origin xyz="0 0 0" rpy="0 0 0" />
       <geometry>
-        <mesh filename="package://libro_model/urdf/meshes/base_link.STL" />
+        <mesh filename="package://libro_model/meshes/base_link.STL" />
       </geometry>
       <material name="">
@@ -35,5 +35,5 @@
       <origin xyz="0 0 0" rpy="0 0 0" />
       <geometry>
-        <mesh filename="package://libro_model/urdf/meshes/base_link.STL" />
+        <mesh filename="package://libro_model/meshes/base_link.STL" />
       </geometry>
     </collision>
@@ -48,14 +48,14 @@
       <origin xyz="0 0 0" rpy="0 0 0" />
       <geometry>
-        <mesh filename="package://libro_model/urdf/meshes/right_front_wheel_link.STL" />
-      </geometry>
-      <material name="">
-        <color rgba="0.298039215686275 0.298039215686275 0.298039215686275 1" />
-      </material>
-    </visual>
-    <collision>
-      <origin xyz="0 0 0" rpy="0 0 0" />
-      <geometry>
-        <mesh filename="package://libro_model/urdf/meshes/right_front_wheel_link.STL" />
+        <mesh filename="package://libro_model/meshes/right_front_wheel_link.STL" />
+      </geometry>
+      <material name="">
+        <color rgba="0.298039215686275 0.298039215686275 0.298039215686275 1" />
+      </material>
+    </visual>
+    <collision>
+      <origin xyz="0 0 0" rpy="0 0 0" />
+      <geometry>
+        <mesh filename="package://libro_model/meshes/right_front_wheel_link.STL" />
       </geometry>
     </collision>
@@ -77,14 +77,14 @@
       <origin xyz="0 0 0" rpy="0 0 0" />
       <geometry>
-        <mesh filename="package://libro_model/urdf/meshes/right_rear_wheel_link.STL" />
-      </geometry>
-      <material name="">
-        <color rgba="0.298039215686275 0.298039215686275 0.298039215686275 1" />
-      </material>
-    </visual>
-    <collision>
-      <origin xyz="0 0 0" rpy="0 0 0" />
-      <geometry>
-        <mesh filename="package://libro_model/urdf/meshes/right_rear_wheel_link.STL" />
+        <mesh filename="package://libro_model/meshes/right_rear_wheel_link.STL" />
+      </geometry>
+      <material name="">
+        <color rgba="0.298039215686275 0.298039215686275 0.298039215686275 1" />
+      </material>
+    </visual>
+    <collision>
+      <origin xyz="0 0 0" rpy="0 0 0" />
+      <geometry>
+        <mesh filename="package://libro_model/meshes/right_rear_wheel_link.STL" />
       </geometry>
     </collision>
@@ -106,14 +106,14 @@
       <origin xyz="0 0 0" rpy="0 0 0" />
       <geometry>
-        <mesh filename="package://libro_model/urdf/meshes/left_front_wheel_link.STL" />
-      </geometry>
-      <material name="">
-        <color rgba="0.298039215686275 0.298039215686275 0.298039215686275 1" />
-      </material>
-    </visual>
-    <collision>
-      <origin xyz="0 0 0" rpy="0 0 0" />
-      <geometry>
-        <mesh filename="package://libro_model/urdf/meshes/left_front_wheel_link.STL" />
+        <mesh filename="package://libro_model/meshes/left_front_wheel_link.STL" />
+      </geometry>
+      <material name="">
+        <color rgba="0.298039215686275 0.298039215686275 0.298039215686275 1" />
+      </material>
+    </visual>
+    <collision>
+      <origin xyz="0 0 0" rpy="0 0 0" />
+      <geometry>
+        <mesh filename="package://libro_model/meshes/left_front_wheel_link.STL" />
       </geometry>
     </collision>
@@ -135,14 +135,14 @@
       <origin xyz="0 0 0" rpy="0 0 0" />
       <geometry>
-        <mesh filename="package://libro_model/urdf/meshes/left_rear_wheel_link.STL" />
-      </geometry>
-      <material name="">
-        <color rgba="0.298039215686275 0.298039215686275 0.298039215686275 1" />
-      </material>
-    </visual>
-    <collision>
-      <origin xyz="0 0 0" rpy="0 0 0" />
-      <geometry>
-        <mesh filename="package://libro_model/urdf/meshes/left_rear_wheel_link.STL" />
+        <mesh filename="package://libro_model/meshes/left_rear_wheel_link.STL" />
+      </geometry>
+      <material name="">
+        <color rgba="0.298039215686275 0.298039215686275 0.298039215686275 1" />
+      </material>
+    </visual>
+    <collision>
+      <origin xyz="0 0 0" rpy="0 0 0" />
+      <geometry>
+        <mesh filename="package://libro_model/meshes/left_rear_wheel_link.STL" />
       </geometry>
     </collision>
@@ -164,5 +164,5 @@
       <origin xyz="0 0 0" rpy="0 0 0" />
       <geometry>
-        <mesh filename="package://libro_model/urdf/meshes/ydlidar_link.STL" />
+        <mesh filename="package://libro_model/meshes/ydlidar_link.STL" />
       </geometry>
       <material name="">
@@ -173,5 +173,5 @@
       <origin xyz="0 0 0" rpy="0 0 0" />
       <geometry>
-        <mesh filename="package://libro_model/urdf/meshes/ydlidar_link.STL" />
+        <mesh filename="package://libro_model/meshes/ydlidar_link.STL" />
       </geometry>
     </collision>
@@ -192,5 +192,5 @@
       <origin xyz="0 0 0" rpy="0 0 0" />
       <geometry>
-        <mesh filename="package://libro_model/urdf/meshes/lidar_underframe_link.STL" />
+        <mesh filename="package://libro_model/meshes/lidar_underframe_link.STL" />
       </geometry>
       <material name="">
@@ -201,5 +201,5 @@
       <origin xyz="0 0 0" rpy="0 0 0" />
       <geometry>
-        <mesh filename="package://libro_model/urdf/meshes/lidar_underframe_link.STL" />
+        <mesh filename="package://libro_model/meshes/lidar_underframe_link.STL" />
       </geometry>
     </collision>
@@ -211,3 +211,84 @@
     <axis xyz="0 0 0" />
   </joint>
+    <link name="camera_link">
+    <inertial>
+      <origin xyz="-0.00303115254709119 9.98333360424652E-16 -5.12569483805715E-05" rpy="0 0 0" />
+      <mass value="0.00145671307075292" />
+      <inertia ixx="6.93646665527772E-08" ixy="3.04630454817989E-24" ixz="-1.09673943150479E-10" iyy="3.98881873637141E-08" iyz="-9.33337790838574E-24" izz="3.98920145491929E-08" />
+    </inertial>
+    <visual>
+      <origin xyz="0 0 0" rpy="0 0 0" />
+      <geometry>
+        <mesh filename="package://libro_model/meshes/camera_link.STL" />
+      </geometry>
+      <material name="">
+        <color rgba="1 1 1 1" />
+      </material>
+    </visual>
+    <collision>
+      <origin xyz="0 0 0" rpy="0 0 0" />
+      <geometry>
+        <mesh filename="package://libro_model/meshes/camera_link.STL" />
+      </geometry>
+    </collision>
+  </link>
+  <joint name="camera_joint" type="fixed">
+    <origin xyz="0.12531 -0.00043191 -0.023" rpy="0 0 0" />
+    <parent link="libro_chassis_link" />
+    <child link="camera_link" />
+    <axis xyz="0 1 0" />
+  </joint>
+    <link
+    name="imu_link">
+    <inertial>
+      <origin
+        xyz="1.38777878078145E-17 -1.76569405348702E-20 0.000480459453048733"
+        rpy="0 0 0" />
+      <mass
+        value="0.00505378695593601" />
+      <inertia
+        ixx="1.40522552943832E-07"
+        ixy="2.7306391434977E-40"
+        ixz="-2.54746894131233E-40"
+        iyy="1.40522552943832E-07"
+        iyz="-1.06659580591594E-25"
+        izz="2.51063192322412E-07" />
+    </inertial>
+    <visual>
+      <origin
+        xyz="0 0 0"
+        rpy="0 0 0" />
+      <geometry>
+        <mesh
+          filename="package://libro_model/meshes/imu_link.STL" />
+      </geometry>
+      <material
+        name="">
+        <color
+          rgba="0.898039215686275 0.917647058823529 0.929411764705882 1" />
+      </material>
+    </visual>
+    <collision>
+      <origin
+        xyz="0 0 0"
+        rpy="0 0 0" />
+      <geometry>
+        <mesh
+          filename="package://libro_model/meshes/imu_link.STL" />
+      </geometry>
+    </collision>
+  </link>
+  <joint
+    name="imu_joint"
+    type="fixed">
+    <origin
+      xyz="0.099307 -1.2058E-05 -0.0305"
+      rpy="0 0 0" />
+    <parent
+      link="libro_chassis_link" />
+    <child
+      link="imu_link" />
+    <axis
+      xyz="0 0 1" />
+  </joint>
 </robot>
