Commit message: 添加了IMU和摄像头
Co-Authored-By: Damongzx <77727892+Damongzx@users.noreply.github.com>
Co-Authored-By: john1217 <13514609+john1217@users.noreply.github.com>

File: libro_model/urdf/libro_model.urdf.xacro (robot description, xacro)
@@ -26,5 +26,5 @@
       <origin xyz="0 0 0" rpy="0 0 0" />
       <geometry>
-        <mesh filename="package://libro_model/urdf/meshes/base_link.STL" />
+        <mesh filename="package://libro_model/meshes/base_link.STL" />
       </geometry>
       <material name="">
@@ -35,5 +35,5 @@
       <origin xyz="0 0 0" rpy="0 0 0" />
       <geometry>
-        <mesh filename="package://libro_model/urdf/meshes/base_link.STL" />
+        <mesh filename="package://libro_model/meshes/base_link.STL" />
       </geometry>
     </collision>
@@ -48,14 +48,14 @@
       <origin xyz="0 0 0" rpy="0 0 0" />
       <geometry>
-        <mesh filename="package://libro_model/urdf/meshes/right_front_wheel_link.STL" />
-      </geometry>
-      <material name="">
-        <color rgba="0.298039215686275 0.298039215686275 0.298039215686275 1" />
-      </material>
-    </visual>
-    <collision>
-      <origin xyz="0 0 0" rpy="0 0 0" />
-      <geometry>
-        <mesh filename="package://libro_model/urdf/meshes/right_front_wheel_link.STL" />
+        <mesh filename="package://libro_model/meshes/right_front_wheel_link.STL" />
+      </geometry>
+      <material name="">
+        <color rgba="0.298039215686275 0.298039215686275 0.298039215686275 1" />
+      </material>
+    </visual>
+    <collision>
+      <origin xyz="0 0 0" rpy="0 0 0" />
+      <geometry>
+        <mesh filename="package://libro_model/meshes/right_front_wheel_link.STL" />
       </geometry>
     </collision>
@@ -77,14 +77,14 @@
       <origin xyz="0 0 0" rpy="0 0 0" />
       <geometry>
-        <mesh filename="package://libro_model/urdf/meshes/right_rear_wheel_link.STL" />
-      </geometry>
-      <material name="">
-        <color rgba="0.298039215686275 0.298039215686275 0.298039215686275 1" />
-      </material>
-    </visual>
-    <collision>
-      <origin xyz="0 0 0" rpy="0 0 0" />
-      <geometry>
-        <mesh filename="package://libro_model/urdf/meshes/right_rear_wheel_link.STL" />
+        <mesh filename="package://libro_model/meshes/right_rear_wheel_link.STL" />
+      </geometry>
+      <material name="">
+        <color rgba="0.298039215686275 0.298039215686275 0.298039215686275 1" />
+      </material>
+    </visual>
+    <collision>
+      <origin xyz="0 0 0" rpy="0 0 0" />
+      <geometry>
+        <mesh filename="package://libro_model/meshes/right_rear_wheel_link.STL" />
       </geometry>
     </collision>
@@ -106,14 +106,14 @@
       <origin xyz="0 0 0" rpy="0 0 0" />
       <geometry>
-        <mesh filename="package://libro_model/urdf/meshes/left_front_wheel_link.STL" />
-      </geometry>
-      <material name="">
-        <color rgba="0.298039215686275 0.298039215686275 0.298039215686275 1" />
-      </material>
-    </visual>
-    <collision>
-      <origin xyz="0 0 0" rpy="0 0 0" />
-      <geometry>
-        <mesh filename="package://libro_model/urdf/meshes/left_front_wheel_link.STL" />
+        <mesh filename="package://libro_model/meshes/left_front_wheel_link.STL" />
+      </geometry>
+      <material name="">
+        <color rgba="0.298039215686275 0.298039215686275 0.298039215686275 1" />
+      </material>
+    </visual>
+    <collision>
+      <origin xyz="0 0 0" rpy="0 0 0" />
+      <geometry>
+        <mesh filename="package://libro_model/meshes/left_front_wheel_link.STL" />
       </geometry>
     </collision>
@@ -135,14 +135,14 @@
       <origin xyz="0 0 0" rpy="0 0 0" />
       <geometry>
-        <mesh filename="package://libro_model/urdf/meshes/left_rear_wheel_link.STL" />
-      </geometry>
-      <material name="">
-        <color rgba="0.298039215686275 0.298039215686275 0.298039215686275 1" />
-      </material>
-    </visual>
-    <collision>
-      <origin xyz="0 0 0" rpy="0 0 0" />
-      <geometry>
-        <mesh filename="package://libro_model/urdf/meshes/left_rear_wheel_link.STL" />
+        <mesh filename="package://libro_model/meshes/left_rear_wheel_link.STL" />
+      </geometry>
+      <material name="">
+        <color rgba="0.298039215686275 0.298039215686275 0.298039215686275 1" />
+      </material>
+    </visual>
+    <collision>
+      <origin xyz="0 0 0" rpy="0 0 0" />
+      <geometry>
+        <mesh filename="package://libro_model/meshes/left_rear_wheel_link.STL" />
       </geometry>
     </collision>
@@ -164,5 +164,5 @@
       <origin xyz="0 0 0" rpy="0 0 0" />
       <geometry>
-        <mesh filename="package://libro_model/urdf/meshes/ydlidar_link.STL" />
+        <mesh filename="package://libro_model/meshes/ydlidar_link.STL" />
       </geometry>
       <material name="">
@@ -173,5 +173,5 @@
       <origin xyz="0 0 0" rpy="0 0 0" />
       <geometry>
-        <mesh filename="package://libro_model/urdf/meshes/ydlidar_link.STL" />
+        <mesh filename="package://libro_model/meshes/ydlidar_link.STL" />
       </geometry>
     </collision>
@@ -192,5 +192,5 @@
       <origin xyz="0 0 0" rpy="0 0 0" />
       <geometry>
-        <mesh filename="package://libro_model/urdf/meshes/lidar_underframe_link.STL" />
+        <mesh filename="package://libro_model/meshes/lidar_underframe_link.STL" />
       </geometry>
       <material name="">
@@ -201,5 +201,5 @@
       <origin xyz="0 0 0" rpy="0 0 0" />
       <geometry>
-        <mesh filename="package://libro_model/urdf/meshes/lidar_underframe_link.STL" />
+        <mesh filename="package://libro_model/meshes/lidar_underframe_link.STL" />
       </geometry>
     </collision>
@@ -211,5 +211,5 @@
     <axis xyz="0 0 0" />
   </joint>
-  <link name="camera_link">
+    <link name="camera_link">
     <inertial>
       <origin xyz="-0.00303115254709119 9.98333360424652E-16 -5.12569483805715E-05" rpy="0 0 0" />
@@ -220,5 +220,5 @@
       <origin xyz="0 0 0" rpy="0 0 0" />
       <geometry>
-        <mesh filename="package://libro_model/urdf/meshes/camera_link.STL" />
+        <mesh filename="package://libro_model/meshes/camera_link.STL" />
       </geometry>
       <material name="">
@@ -229,5 +229,5 @@
       <origin xyz="0 0 0" rpy="0 0 0" />
       <geometry>
-        <mesh filename="package://libro_model/urdf/meshes/camera_link.STL" />
+        <mesh filename="package://libro_model/meshes/camera_link.STL" />
       </geometry>
     </collision>
@@ -239,16 +239,56 @@
     <axis xyz="0 1 0" />
   </joint>
-  <link name="imu_link">
-    <visual>
-      <geometry>
-        <box size="0.01 0.01 0.01"/>
-      </geometry>
-    </visual>
-  </link>
-  <joint name="imu_joint" type="fixed">
-    <origin xyz="0 0 0.01" rpy="0 0 0" />
-    <parent link="libro_chassis_link" />
-    <child link="imu_link" />
-    <axis xyz="0 0 0" />
+    <link
+    name="imu_link">
+    <inertial>
+      <origin
+        xyz="1.38777878078145E-17 -1.76569405348702E-20 0.000480459453048733"
+        rpy="0 0 0" />
+      <mass
+        value="0.00505378695593601" />
+      <inertia
+        ixx="1.40522552943832E-07"
+        ixy="2.7306391434977E-40"
+        ixz="-2.54746894131233E-40"
+        iyy="1.40522552943832E-07"
+        iyz="-1.06659580591594E-25"
+        izz="2.51063192322412E-07" />
+    </inertial>
+    <visual>
+      <origin
+        xyz="0 0 0"
+        rpy="0 0 0" />
+      <geometry>
+        <mesh
+          filename="package://libro_model/meshes/imu_link.STL" />
+      </geometry>
+      <material
+        name="">
+        <color
+          rgba="0.898039215686275 0.917647058823529 0.929411764705882 1" />
+      </material>
+    </visual>
+    <collision>
+      <origin
+        xyz="0 0 0"
+        rpy="0 0 0" />
+      <geometry>
+        <mesh
+          filename="package://libro_model/meshes/imu_link.STL" />
+      </geometry>
+    </collision>
+  </link>
+  <joint
+    name="imu_joint"
+    type="fixed">
+    <origin
+      xyz="0.099307 -1.2058E-05 -0.0305"
+      rpy="0 0 0" />
+    <parent
+      link="libro_chassis_link" />
+    <child
+      link="imu_link" />
+    <axis
+      xyz="0 0 1" />
   </joint>
 </robot>

Commit message: merge and update imu-issue to dev

File: libro_model/urdf/libro_model.urdf.xacro (robot description, xacro)
@@ -211,5 +211,5 @@
     <axis xyz="0 0 0" />
   </joint>
-  <link name="camera_link">
+    <link name="camera_link">
     <inertial>
       <origin xyz="-0.00303115254709119 9.98333360424652E-16 -5.12569483805715E-05" rpy="0 0 0" />
